File: SharpMem_Grid.sch (KiCad schematic (older format))
At the start: 28 parts

Commit message: Annotated and associated footprints
Parts:
- C1, C2, C3, C4, C5, C6, C7: renamed from C?; footprint (none) -> Capacitors_SMD:C_0603
- P1: renamed from P?; footprint (none) -> Solutions:USB_B_VERTICAL
- P2: renamed from P?; footprint (none) -> Pin_Headers:Pin_Header_Straight_2x04_Pitch2.54mm
- R1, R10, R11, R12, R2, R3, R4, R5, R6, R7, R8, R9: renamed from R?; footprint (none) -> Capacitors_SMD:C_0603
- SW1, SW2: renamed from SW?; footprint (none) -> OpenBCI:PTS810
- U1: renamed from U?; footprint (none) -> Housings_SOIC:SOIJ-8_5.3x5.3mm_Pitch1.27mm
- U3: renamed from U?; value PIC32MX250F128B -> PIC32MX250F128B-I/SS; footprint (none) -> Housings_SSOP:SSOP-28_5.3x10.2mm_Pitch0.65mm
- Y1: renamed from Y?; footprint (none) -> Solutions:ABLS_SMT_XTAL
- gave numbers to parts that had none: 2
Other:
- note added: "25LC1024T-I/SM\n"
- note removed: "25LC1024X_X_SM"

Commit message: Moved Library and updated paths
Parts:
- SW1, SW2: footprint OpenBCI:PTS810 -> Solutions:PTS810
Changed lines of the file:
@@
 EESchema Schematic File Version 2
-LIBS:Solutions
-LIBS:Tympan
 LIBS:power
 LIBS:device
@@
 LIBS:contrib
 LIBS:valves
-LIBS:OpenBCI
+LIBS:Solutions
 LIBS:SharpMem_Grid-cache
 EELAYER 25 0
@@
 F 0 "SW2" H 2300 6910 50  0000 C CNN
 F 1 "PTS810_SJK_250_SMTR_LFS" H 2150 6600 50  0000 C CNN
-F 2 "OpenBCI:PTS810" H 2150 6800 50  0001 C CNN
+F 2 "Solutions:PTS810" H 2150 6800 50  0001 C CNN
 F 3 "" H 2150 6800 50  0000 C CNN
 	1    2150 6800
@@
 F 0 "SW1" H 2000 4550 50  0000 C CNN
 F 1 "PTS810_SJK_250_SMTR_LFS" H 1950 4900 50  0000 C CNN
-F 2 "OpenBCI:PTS810" H 2100 4750 50  0001 C CNN
+F 2 "Solutions:PTS810" H 2100 4750 50  0001 C CNN
 F 3 "" H 2100 4750 50  0000 C CNN
 	1    2100 4750

Commit message: Laid out the schematic
Parts:
- P1: symbol USB_B -> USB_B-RESCUE-SharpMem_Grid
Other:
- note added: "PCB 1.25X1.375"
Changed lines of the file:
@@
 EESchema Schematic File Version 2
+LIBS:SharpMem_Grid-rescue
 LIBS:power
 LIBS:device
@@
 	1    0    0    -1
 $EndComp
+Text Label 7400 4350 2    60   ~ 0
+MOSI
 Text Label 7400 4250 2    60   ~ 0
-MOSI
-Text Label 7400 4350 2    60   ~ 0
 SCLK
 Text Label 7400 4450 2    60   ~ 0
@@
 MOSI
 $Comp
-L USB_B P1
+L USB_B-RESCUE-SharpMem_Grid P1
 U 1 1 5B8487E7
 P 2600 2300
@@
 	5700 4650 5700 4850
 Connection ~ 5400 4850
+Text Notes 3750 3450 0    60   ~ 0
+PCB 1.25X1.375
 $EndSCHEMATC

Commit message: ASSOCIATED FOOTPRINTS
Parts:
- DIS1: footprint (none) -> Solutions:MOLEX_505110-1092
- U2: footprint (none) -> Solutions:SSOP-5-0.65_PITCH
Changed lines of the file:
@@
 F 0 "DIS1" H 8850 2650 60  0000 C CNN
 F 1 "SharpMem_LCD_96x96" H 9200 3950 60  0000 C CNN
-F 2 "" H 8500 4050 60  0001 C CNN
+F 2 "Solutions:MOLEX_505110-1092" H 8500 4050 60  0001 C CNN
 F 3 "" H 8500 4050 60  0000 C CNN
 	1    8500 4050
@@
 F 0 "U2" H 7375 2225 60  0000 C CNN
 F 1 "Schmitt_Inverter_Single" H 8450 2250 60  0000 C CNN
-F 2 "" H 7900 2350 60  0001 C CNN
+F 2 "Solutions:SSOP-5-0.65_PITCH" H 7900 2350 60  0001 C CNN
 F 3 "" H 7900 2350 60  0000 C CNN
 	1    7900 2350

Commit message: Lay out components
Parts:
- added D1: LED, Capacitors_SMD:C_0603, symbol LED
- added J1: CONN_01X05, Pin_Headers:Pin_Header_Straight_1x05_Pitch2.00mm, symbol CONN_01X05
- added R13: 10K, Capacitors_SMD:C_0603, symbol R
Connections:
- net +3V3: now also J1.2 (P2)
- net EE_SS: now also U3.2 (RA0); no longer U3.4 (RB0)
- net GND: now also J1.3 (P3), R13.1
- net LCD_SS: now also U3.6 (RB2); no longer U3.5 (RB1)
- net MCLR: now also J1.1 (P1)
- net LED: now reaches U3.7 (RB2)
- net LED: now also D1.2 (A)
- new net: D1.1 (K), R13.2
- new net PGC: J1.5 (P5), U3.5 (RB1)
- new net PGD: J1.4 (P4), U3.4 (RB0)
Other:
- note removed: "PCB 1.25X1.375"
- moved on the sheet: C5, C6, C7, R12, R6, SW1, SW2, U3, Y1

Commit message: Routed traces and copper pour. Passes DFM
Connections:
- net DISP: now also U3.17 (RB8); no longer U3.26 (RB15)
- net EE_SS: now also U3.6 (RB2); no longer U3.2 (RA0)
- net LCD_SS: now also U3.16 (RB7); no longer U3.6 (RB2)
Changed lines of the file:
@@
 Text Label 2550 4550 2    60   ~ 0
 MISO
-Text Label 2550 4450 2    60   ~ 0
+Text Label 2550 4850 2    60   ~ 0
 EE_SS
-Text Label 2550 4850 2    60   ~ 0
+Text Label 3900 4550 0    60   ~ 0
 LCD_SS
 Text Label 3900 4950 0    60   ~ 0
@@
 Text Label 3900 5150 0    60   ~ 0
 SCLK
-Text Label 3900 5250 0    60   ~ 0
+Text Label 3900 4650 0    60   ~ 0
 DISP
 Text Label 3900 4350 0    60   ~ 0

Commit message: Final layout and BOM
Parts:
- added J2, J3: CONN_01X01, Solutions:NPT_125mil, symbol CONN_01X01
- Y1: value ABLS-8.000MHZ-B4-T -> ECS-080-18-23G-JGN-TR; footprint Solutions:ABLS_SMT_XTAL -> Solutions:ECS-080-18-23G-JGN-TR_8MHz_60x35
Changed lines of the file:
@@
 P 1850 5100
 F 0 "Y1" V 1850 4900 50  0000 C CNN
-F 1 "ABLS-8.000MHZ-B4-T" V 1650 4700 50  0000 C CNN
-F 2 "Solutions:ABLS_SMT_XTAL" H 1850 5100 50  0001 C CNN
+F 1 "ECS-080-18-23G-JGN-TR" V 1650 4700 50  0000 C CNN
+F 2 "Solutions:ECS-080-18-23G-JGN-TR_8MHz_60x35" H 1850 5100 50  0001 C CNN
 F 3 "" H 1850 5100 50  0000 C CNN
 	1    1850 5100
@@
 Text Label 2800 7050 2    60   ~ 0
 LED
+$Comp
+L CONN_01X01 J2
+U 1 1 5B8C06B2
+P 3950 1150
+F 0 "J2" H 3950 1250 50  0000 C CNN
+F 1 "CONN_01X01" H 4300 1150 50  0000 C CNN
+F 2 "Solutions:NPT_125mil" H 3950 1150 50  0001 C CNN
+F 3 "" H 3950 1150 50  0001 C CNN
+	1    3950 1150
+	1    0    0    -1
+$EndComp
+$Comp
+L CONN_01X01 J3
+U 1 1 5B8C0716
+P 3950 1300
+F 0 "J3" H 3950 1200 50  0000 C CNN
+F 1 "CONN_01X01" H 4300 1300 50  0000 C CNN
+F 2 "Solutions:NPT_125mil" H 3950 1300 50  0001 C CNN
+F 3 "" H 3950 1300 50  0001 C CNN
+	1    3950 1300
+	1    0    0    -1
+$EndComp
 $EndSCHEMATC
